File: eth2rs485.brd (EAGLE design)
At the start: 31.7 x 86.4 mm, 59 parts, among them IC1 VREG-OKI-78SR-5.0/1.5-W36, IC2 MAX485, IC3 24AA025E48, T1 74990101217, U1 AP2112, U2 ATMEGA644P-20AU, U3 W5500, Y1 IT-L30-010, Y2 CSTCE16M0V53-R0 16MHZ

Commit message: atmega 644 working (hopefully)
Parts:
- removed U$1: (no value), logo:CE_5MM
- C3: value 1µF -> 10uF
- C6: value 2.2µF -> 10uF
Other:
- board text added: "90040-V0.2"
- board text added: "Ethernet RS485 Bridge V0.2"
- board text added: "codm.de 2019"
- board text removed: "90040-V0.1"
- board text removed: "Ethernet RS485 Bridge V0.4"
- board text removed: "codm.de (c) 2019"
Changed lines of the file:
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@@
 <?xml version="1.0" encoding="utf-8"?>
 <!DOCTYPE eagle SYSTEM "eagle.dtd">
-<eagle version="9.3.0">
+<eagle version="9.3.1">
 <drawing>
 <settings>
@@
 <layer number="20" name="Dimension" color="24" fill="1" visible="yes" active="yes"/>
 <layer number="21" name="tPlace" color="7" fill="1" visible="yes" active="yes"/>
-<layer number="22" name="bPlace" color="7" fill="1" visible="no" active="yes"/>
+<layer number="22" name="bPlace" color="7" fill="1" visible="yes" active="yes"/>
 <layer number="23" name="tOrigins" color="15" fill="1" visible="yes" active="yes"/>
 <layer number="24" name="bOrigins" color="15" fill="1" visible="yes" active="yes"/>
@@
 DMX-</text>
 <text x="15.8" y="60.25" size="1.778" layer="26" font="vector" ratio="10" rot="MR180" align="center">Ethernet RS485
-Bridge V0.4</text>
+Bridge V0.2</text>
 <wire x1="0" y1="23.15" x2="32" y2="23.15" width="0.127" layer="150"/>
 <wire x1="0" y1="63.3" x2="32" y2="63.3" width="0.1016" layer="150"/>
@@
 <wire x1="1.55" y1="42.4" x2="1.55" y2="44" width="0.127" layer="150"/>
 <wire x1="30.15" y1="42.4" x2="30.15" y2="44" width="0.127" layer="150"/>
-<text x="15.85" y="18.35" size="1.27" layer="25" font="vector" ratio="10" distance="40" rot="R180" align="center">codm.de (c) 2019</text>
+<text x="15.85" y="18.35" size="1.27" layer="25" font="vector" ratio="10" distance="40" rot="R180" align="center">codm.de 2019</text>
 <text x="7" y="20" size="1.778" layer="27" font="vector">5V FOCA</text>
 <text x="10.15" y="12.4" size="0.8" layer="25" font="vector">5V</text>
-<text x="29.15" y="43.3" size="1.778" layer="26" font="vector" rot="MR270" align="bottom-center">90040-V0.1</text>
+<text x="29.15" y="43.3" size="1.778" layer="26" font="vector" rot="MR270" align="bottom-center">90040-V0.2</text>
 <rectangle x1="-0.00126875" y1="-0.00126875" x2="0.575309375" y2="0.00126875" layer="201"/>
 <rectangle x1="-0.00126875" y1="0.00126875" x2="0.575309375" y2="0.003809375" layer="201"/>
@@
 <attribute name="VALUE" x="6.36" y="47.36" size="0.8" layer="27"/>
 </element>
-<element name="C3" library="rcl" library_urn="urn:adsk.eagle:library:334" package="C0805" package3d_urn="urn:adsk.eagle:package:23617/2" value="1µF" x="28.3" y="51" smashed="yes" rot="R180">
+<element name="C3" library="rcl" library_urn="urn:adsk.eagle:library:334" package="C0805" package3d_urn="urn:adsk.eagle:package:23617/2" value="10uF" x="28.3" y="51" smashed="yes" rot="R180">
 <attribute name="NAME" x="28.3" y="49.8646" size="0.7" layer="25" font="vector" align="top-center"/>
 <attribute name="SPICEPREFIX" value="C" x="28.3" y="51" size="1.778" layer="27" rot="R180" display="off"/>
 <attribute name="VALUE" x="29.9" y="53.1" size="1.016" layer="27" rot="R180"/>
 </element>
-<element name="C6" library="rcl" library_urn="urn:adsk.eagle:library:334" package="C0805" package3d_urn="urn:adsk.eagle:package:23617/2" value="2.2µF" x="28.3" y="56.45" smashed="yes" rot="R180">
+<element name="C6" library="rcl" library_urn="urn:adsk.eagle:library:334" package="C0805" package3d_urn="urn:adsk.eagle:package:23617/2" value="10uF" x="28.3" y="56.45" smashed="yes" rot="R180">
 <attribute name="NAME" x="28.3" y="57.5854" size="0.7" layer="25" font="vector" align="bottom-center"/>
 <attribute name="SPICEPREFIX" value="C" x="28.3" y="56.45" size="1.778" layer="27" rot="R180" display="off"/>
@@
 <attribute name="NAME" x="4.1" y="18.85" size="0.7" layer="21" font="vector" align="center"/>
 </element>
-<element name="U$1" library="logo" library_urn="urn:adsk.eagle:library:264" package="CE_5MM" value="" x="15" y="32" smashed="yes" rot="MR0"/>
 <element name="LOGO2" library="SparkFun-Aesthetics" package="OSHW-LOGO-M" value="OSHW-LOGOM" x="15.8" y="41" smashed="yes" rot="MR0"/>
 <element name="U$3" library="codm" package="WEEE-LOGO-8MM" value="" x="24.8837" y="25.1887" smashed="yes" rot="MR0"/>

Commit message: added sch pdf, minor changes brd
Parts:
- C10, C13: value 0.1uF -> 100nF
- C15: device rcl:R0805 -> rcl:C0805
- R1: value 220 -> 2k7
- X1: value (none) -> MSTBA3; device con-ptr500:AK500/3 -> con-phoenix-508:MSTBA3
- X2: value (none) -> MSTBA2; device con-ptr500:AK500/2 -> con-phoenix-508:MSTBA2
- moved F1 25.5 mm to (2.70, 27.4)
- moved D1 5.32 mm to (4.10, 32.8), turned to 0 degrees
- moved X1 3.52 mm to (22.8, 0.50)
- moved X2 3.47 mm to (6.30, 0.50)
- moved ISP 1.24 mm to (4.40, 38.0)
- moved Y1 0.32 mm to (8.80, 43.9)
- moved R10 0.32 mm to (5.30, 44.8)
- moved C8 0.32 mm to (3.10, 44.8)
- moved C7 0.32 mm to (14.6, 44.8)
- moved R8 0.32 mm to (12.4, 44.8)
- moved IC3 0.30 mm to (11.6, 35.0)
- moved IC1 0.22 mm to (9.55, 26.4)
- moved Y2 0.20 mm to (14.6, 40.0)
Routing:
- net N$8: track 29.8 -> 9.73 mm
- net VCC: track 6.21 -> 21.8 mm
- net +5V: track 99.9 -> 109.5 mm, vias 3 -> 2
- net RST: track 93.6 -> 90.6 mm
- net N$11: track 19.2 -> 17.7 mm
- net N$4: track 22.5 -> 21.2 mm
- net N$6: track 21.3 -> 20.0 mm
- net N$5: track 23.6 -> 22.7 mm
- net MOSI: track 36.1 -> 35.3 mm, vias 2 -> 3
- net SCL: track 13.9 -> 14.5 mm
- net MISO: track 37.3 -> 37.2 mm, vias 2 -> 3
Other:
- board text added: "1"
- board text added: "90040-V0.3"
- board text added: "Ethernet RS485 Bridge V0.3"
- board text added: "codm.de 2020"
- board text added: "codm.de 2020 CC-BY-SA-NC"
- board text removed: "90040-V0.2"
- board text removed: "Ethernet RS485 Bridge V0.2"
- board text removed: "codm.de 2019"
- board text removed: "codm.de 2019 CC-BY-SA"
